File: examples/two_die_interposer/kicad/two_die_interposer.kicad_sch (KiCad schematic)
At the start: 37 parts, among them J10 IOPad_WireBond_100x100, J12 IOPad_WireBond_100x100, J13 IOPad_WireBond_100x100, J14 IOPad_WireBond_100x100, J15 IOPad_WireBond_100x100, J16 IOPad_WireBond_100x100, J17 IOPad_WireBond_100x100, J18 IOPad_WireBond_100x100, J19 IOPad_WireBond_100x100, J2 IOPad_WireBond_100x100, J20 IOPad_WireBond_100x100, J21 IOPad_WireBond_100x100, J22 IOPad_WireBond_100x100, J23 IOPad_WireBond_100x100, J24 IOPad_WireBond_100x100, J25 IOPad_WireBond_100x100, J26 IOPad_WireBond_100x100, J27 IOPad_WireBond_100x100, J28 IOPad_WireBond_100x100, J29 IOPad_WireBond_100x100, J3 IOPad_WireBond_100x100, J30 IOPad_WireBond_100x100, J31 IOPad_WireBond_100x100, J32 IOPad_WireBond_100x100, J33 IOPad_WireBond_100x100, J34 IOPad_WireBond_100x100, J35 IOPad_WireBond_100x100, J36 IOPad_WireBond_100x100, J37 IOPad_WireBond_100x100, J39 IOPad_WireBond_100x100, J40 IOPad_WireBond_100x100, J41 IOPad_WireBond_100x100, J42 IOPad_WireBond_100x100, J43 IOPad_WireBond_100x100, J9 IOPad_WireBond_100x100, U1 Metal_Test, U2 Metal_Test

Commit message: Make two_die_interposer footprint reproducible from a shipped stripped GDS
Ship chiplets/Metal_Test_stripped.gds: the curated die layout (only the 58 I/O
pads on 134/0, names on 134/25), the frozen result of the human-in-the-loop pad
review. metal_test_chiplet's footprint now regenerates one-shot from it with no
manual KLayout step, reproducing the committed footprint exactly.

Align the two power pads to the die's real 134/25 label VCC (they were Vcc)
across the footprint, symbol, pin list, board and schematic, so the committed
library matches its own source die. Connectivity is unchanged (net codes keep
their pad bindings; the user net stays vcc), and the assembly GDS/.chiplet and
DRC are byte-identical since pad names do not reach the assembly outputs; only
U2's two auto-generated no-connect placeholder net names track the rename.

Ship chiplets/metal_test_chiplet.g2kproj too: a saved gds-to-kicad GUI session
(input + stripped GDS, LYP, layer selections and the embedded pin list) so
"gds-to-kicad -> File -> Open Project" lands at the exact state that produces the
footprint and symbol. It stores image-absolute paths, for use in the container.

verify gate (adk-verify-chiplet-artifacts): step 4 regenerates the footprint from
the shipped stripped GDS and asserts its pad set equals the committed one exactly
(name + shape + position + size + layers + custom-pad gr_poly outline); step 5 is
the former full-GDS liveness smoke; step 6 checks the .g2kproj format, layer
selections and that its embedded pin list matches the shipped pins.json.

Update chiplets/README.md and CHANGELOG.
Connections:
- net vcc: now also U1.VCC; no longer U1.Vcc
Changed lines of the file:
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@@
 		(pin "PA_Vcc4"
 		)
-		(pin "Vcc"
+		(pin "VCC"
 		)
 		(pin "NC"
@@
 		(pin "NC"
 		)
-		(pin "Vcc"
+		(pin "VCC"
 		)
 		(pin "NC"
@@
 		(pin "PA_Vcc4"
 		)
-		(pin "Vcc"
+		(pin "VCC"
 		)
 		(pin "NC"
@@
 		(pin "NC"
 		)
-		(pin "Vcc"
-		)
-		(pin "NC"
+		(pin "VCC"
+		)
+		(pin "NC"
